File: proyecto_desarrollo.kicad_pcb (KiCad board)
At the start: 4 copper layers, 100.2 x 100.2 mm, 47 parts, among them J1 USB_B, J2 UART, Q1 MMBT3904, SW1 SW_SPST, SW2 SW_SPST, SW3 SW_SPST, U1 NE555D, U2 NE555D, U3 4040, U4 4040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

Commit message: Add files via upload
Parts:
- moved R4 2.79 mm to (182.6, 94.1)
- moved C5 2.79 mm to (178.2, 84.7)
- moved C6 2.79 mm to (187.7, 89.0)
- moved U2 2.79 mm to (182.0, 88.7)
- moved G*** 0.84 mm to (123.4, 99.4)
Routing:
- net (no net): track 8.01 -> 0.00 mm
- net +5V: track 251.3 -> 247.0 mm, vias 8 -> 7
- net Net-(U2-DIS): track 21.7 -> 18.9 mm
- net Net-(U2-Q): track 13.7 -> 16.0 mm
- net /alarm: track 34.4 -> 35.2 mm

Commit message: Add files via upload
Routing:
- net Net-(SW1-B): track 138.1 -> 123.9 mm
- net +5V: track 247.0 -> 237.3 mm
- net /alarm: track 35.2 -> 30.9 mm
- net GND: track 55.6 -> 59.3 mm
- net Net-(U2-Q): track 16.0 -> 12.7 mm
- net Net-(BZ1--): track 14.0 -> 14.8 mm
- net /reset: track 59.7 -> 60.3 mm
- added copper zone on In2.Cu, net GND

Commit message: Add files via upload
Parts:
- removed the G*** at (123.4, 99.4)
- added G***: LOGO, footprints:paella2, F.Cu at (129.0, 125.7)
- RV1, RV2: footprint Potentiometer_THT:Potentiometer_ACP_CA6-H2,5_Horizontal -> footprints:601030_AVX
- moved J2 40.2 mm to (175.9, 138.8), turned to -90 degrees
- moved C8 34.2 mm to (185.6, 80.2)
- moved C7 30.5 mm to (151.6, 80.8)
- moved C9 26.6 mm to (172.9, 82.2), turned to 180 degrees
- moved C4 25.1 mm to (182.0, 92.7), turned to 0 degrees
- moved C3 19.7 mm to (156.1, 89.3), turned to 0 degrees
- moved C10 17.0 mm to (184.7, 99.2)
- moved RV2 12.0 mm to (166.4, 104.4), turned to 180 degrees
- moved R4 8.85 mm to (176.1, 88.1)
- moved C11 6.80 mm to (169.7, 102.3), turned to -90 degrees
- moved RV1 5.55 mm to (144.4, 94.8), turned to 90 degrees
- moved U6 4.15 mm to (176.3, 103.6)
- moved R7 3.42 mm to (150.7, 77.9)
- moved R8 3.14 mm to (150.7, 76.4)
- moved R9 2.92 mm to (150.7, 74.9)
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Routing:
- net +5V: track 237.3 -> 334.7 mm, vias 7 -> 13
- net Net-(J2-Pin_1): track 7.92 -> 42.1 mm, vias 0 -> 1
- net Net-(J2-Pin_2): track 7.95 -> 38.6 mm, vias 0 -> 1
- net Net-(U2-DIS): track 18.9 -> 32.1 mm, vias 0 -> 1
- net GND: track 59.3 -> 47.5 mm, vias 14 -> 52
- net Net-(U5-+): track 51.1 -> 45.2 mm
- net /alarm: track 30.9 -> 35.3 mm
- net Net-(U1-DIS): track 14.5 -> 10.8 mm
- net Net-(U3-Q1): track 5.85 -> 2.30 mm
- net Net-(U3-Q2): track 5.54 -> 2.24 mm
- net Net-(U3-Q11): track 5.32 -> 2.19 mm
- net Net-(U3-Q3): track 5.24 -> 2.14 mm
- net Net-(U3-Q5): track 5.02 -> 2.09 mm
- net Net-(U3-Q6): track 4.99 -> 2.15 mm
- net /USB N: track 16.2 -> 19.1 mm
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