File: proyecto_desarrollo.kicad_sch (KiCad schematic)
At the start: 45 parts, among them J1 USB_B, J2 UART, Q1 MMBT3904, SW1 SW_SPST, SW2 SW_SPST, SW3 SW_SPST, U1 NE555D, U2 NE555D, U3 4040, U4 4040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

Commit message: Add files via upload
Parts:
- RV1, RV2: footprint Potentiometer_THT:Potentiometer_ACP_CA6-H2,5_Horizontal -> footprints:601030_AVX
Changed lines of the file:
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@@
 			)
 		)
-		(property "Footprint" "Potentiometer_THT:Potentiometer_ACP_CA6-H2,5_Horizontal"
+		(property "Footprint" "footprints:601030_AVX"
 			(at 86.36 46.99 0)
 			(effects
@@
 			)
 		)
-		(property "Footprint" "Potentiometer_THT:Potentiometer_ACP_CA6-H2,5_Horizontal"
+		(property "Footprint" "footprints:601030_AVX"
 			(at 176.53 46.99 0)
 			(effects
